Commit message: Add and update lot of stuff

File: urdf/ant.urdf (robot description, URDF)
Before this commit: robot object, 1 links, 0 joints
Links:
- added link Abdomen, mass 0; collision mesh filename=package://animals_description/meshes/ant/Abdomen.stl; visual mesh filename=package://animals_description/meshes/ant/Abdomen.stl
- added link Head, mass 4.2276; collision mesh filename=package://animals_description/meshes/ant/Skull.stl; visual mesh filename=package://animals_description/meshes/ant/Skull.stl
- added link HeadLAntenaFoot_J1
- added link HeadLAntenaFoot_J2
- added link HeadLAntena_J1
- added link HeadLAntena_J2
- added link HeadRAntenaFoot_J1
- added link HeadRAntenaFoot_J2
- added link HeadRAntena_J1
- added link HeadRAntena_J2
- added link LAntena, mass 1; collision mesh filename=package://animals_description/meshes/ant/LAntena.stl; visual mesh filename=package://animals_description/meshes/ant/LAntena.stl
- added link LAntenaFoot, mass 1; collision mesh filename=package://animals_description/meshes/ant/LAntenaFoot.stl; visual mesh filename=package://animals_description/meshes/ant/LAntenaFoot.stl
- added link LBFoot, mass 1; collision mesh filename=package://animals_description/meshes/ant/LBFoot.stl; visual mesh filename=package://animals_description/meshes/ant/LBFoot.stl
- added link LBFootSphere; collision sphere radius=0.005; visual sphere radius=0.005
- added link LBShank, mass 1; collision mesh filename=package://animals_description/meshes/ant/LBShank.stl; visual mesh filename=package://animals_description/meshes/ant/LBShank.stl
- added link LBThigh, mass 1; collision mesh filename=package://animals_description/meshes/ant/LBThigh.stl; visual mesh filename=package://animals_description/meshes/ant/LBThigh.stl
- added link LFFoot, mass 1; collision mesh filename=package://animals_description/meshes/ant/LFFoot.stl; visual mesh filename=package://animals_description/meshes/ant/LFFoot.stl
- added link LFFootSphere; collision sphere radius=0.005; visual sphere radius=0.005
- added link LFShank, mass 1; collision mesh filename=package://animals_description/meshes/ant/LFShank.stl; visual mesh filename=package://animals_description/meshes/ant/LFShank.stl
- added link LFThigh, mass 1; collision mesh filename=package://animals_description/meshes/ant/LFThigh.stl; visual mesh filename=package://animals_description/meshes/ant/LFThigh.stl
- added link LMFoot, mass 1; collision mesh filename=package://animals_description/meshes/ant/LMFoot.stl; visual mesh filename=package://animals_description/meshes/ant/LMFoot.stl
- added link LMFootSphere; collision sphere radius=0.005; visual sphere radius=0.005
- added link LMShank, mass 1; collision mesh filename=package://animals_description/meshes/ant/LMShank.stl; visual mesh filename=package://animals_description/meshes/ant/LMShank.stl
- added link LMThigh, mass 1; collision mesh filename=package://animals_description/meshes/ant/LMThigh.stl; visual mesh filename=package://animals_description/meshes/ant/LMThigh.stl
- added link RAntena, mass 1; collision mesh filename=package://animals_description/meshes/ant/RAntena.stl; visual mesh filename=package://animals_description/meshes/ant/RAntena.stl
- added link RAntenaFoot, mass 1; collision mesh filename=package://animals_description/meshes/ant/RAntenaFoot.stl; visual mesh filename=package://animals_description/meshes/ant/RAntenaFoot.stl
- added link RBFoot, mass 1; collision mesh filename=package://animals_description/meshes/ant/RBFoot.stl; visual mesh filename=package://animals_description/meshes/ant/RBFoot.stl
- added link RBFootSphere; collision sphere radius=0.005; visual sphere radius=0.005
- added link RBShank, mass 1; collision mesh filename=package://animals_description/meshes/ant/RBShank.stl; visual mesh filename=package://animals_description/meshes/ant/RBShank.stl
- added link RBThigh, mass 1; collision mesh filename=package://animals_description/meshes/ant/RBThigh.stl; visual mesh filename=package://animals_description/meshes/ant/RBThigh.stl
- added link RFFoot, mass 1; collision mesh filename=package://animals_description/meshes/ant/RFFoot.stl; visual mesh filename=package://animals_description/meshes/ant/RFFoot.stl
- added link RFFootSphere; collision sphere radius=0.005; visual sphere radius=0.005
- added link RFShank, mass 1; collision mesh filename=package://animals_description/meshes/ant/RFShank.stl; visual mesh filename=package://animals_description/meshes/ant/RFShank.stl
- added link RFThigh, mass 1; collision mesh filename=package://animals_description/meshes/ant/RFThigh.stl; visual mesh filename=package://animals_description/meshes/ant/RFThigh.stl
- added link RMFoot, mass 1; collision mesh filename=package://animals_description/meshes/ant/RMFoot.stl; visual mesh filename=package://animals_description/meshes/ant/RMFoot.stl
- added link RMFootSphere; collision sphere radius=0.005; visual sphere radius=0.005
- added link RMShank, mass 1; collision mesh filename=package://animals_description/meshes/ant/RMShank.stl; visual mesh filename=package://animals_description/meshes/ant/RMShank.stl
- added link RMThigh, mass 1; collision mesh filename=package://animals_description/meshes/ant/RMThigh.stl; visual mesh filename=package://animals_description/meshes/ant/RMThigh.stl
- added link Thorax, mass 1; collision mesh filename=package://animals_description/meshes/ant/Thorax.stl; visual mesh filename=package://animals_description/meshes/ant/Thorax.stl
- added link ThoraxAbdomen_J1
- added link ThoraxAbdomen_J2
- added link ThoraxHead_J1
- added link ThoraxHead_J2
- added link ThoraxLBFoot_J1
- added link ThoraxLBFoot_J2
- added link ThoraxLBShank_J1
- added link ThoraxLBShank_J2
- added link ThoraxLBThigh_J1
- added link ThoraxLBThigh_J2
- added link ThoraxLFFoot_J1
- added link ThoraxLFFoot_J2
- added link ThoraxLFShank_J1
- added link ThoraxLFShank_J2
- added link ThoraxLFThigh_J1
- added link ThoraxLFThigh_J2
- added link ThoraxLMFoot_J1
- added link ThoraxLMFoot_J2
- added link ThoraxLMShank_J1
- added link ThoraxLMShank_J2
- added link ThoraxLMThigh_J1
- added link ThoraxLMThigh_J2
- added link ThoraxRBFoot_J1
- added link ThoraxRBFoot_J2
- added link ThoraxRBShank_J1
- added link ThoraxRBShank_J2
- added link ThoraxRBThigh_J1
- added link ThoraxRBThigh_J2
- added link ThoraxRFFoot_J1
- added link ThoraxRFFoot_J2
- added link ThoraxRFShank_J1
- added link ThoraxRFShank_J2
- added link ThoraxRFThigh_J1
- added link ThoraxRFThigh_J2
- added link ThoraxRMFoot_J1
- added link ThoraxRMFoot_J2
- added link ThoraxRMShank_J1
- added link ThoraxRMShank_J2
- added link ThoraxRMThigh_J1
- added link ThoraxRMThigh_J2
- link base_link: mass 1.0 -> None; geometry 
Joints:
- added joint Abdomen: type revolute, parent ThoraxAbdomen_J1, child Abdomen, origin xyz=0 0 0 rpy=0 0 0, axis 0 0 1, limit lower=-0.2 upper=0.2 effort=0 velocity=1.0
- added joint Head: type revolute, parent ThoraxHead_J2, child Head, origin xyz=0 0 0 rpy=0 0 0, axis 0 0 1, limit lower=-0.2 upper=0.2 effort=0 velocity=1.0
- added joint HeadLAntenaFoot_J1: type revolute, parent LAntena, child HeadLAntenaFoot_J1, origin xyz=0.0267 -0.0198 0.1006 rpy=0 0 0, axis 1 0 0, limit lower=-0.4 upper=0.4 effort=0 velocity=1.0
- added joint HeadLAntenaFoot_J2: type revolute, parent HeadLAntenaFoot_J1, child HeadLAntenaFoot_J2, origin xyz=0 0 0 rpy=0 0 0, axis 0 1 0, limit lower=-0.4 upper=0.4 effort=0 velocity=1.0
- added joint HeadLAntena_J1: type revolute, parent Head, child HeadLAntena_J1, origin xyz=0.0176 -0.1027 0.0225 rpy=0 0 0, axis 1 0 0, limit lower=-0.4 upper=0.4 effort=0 velocity=1.0
- added joint HeadLAntena_J2: type revolute, parent HeadLAntena_J1, child HeadLAntena_J2, origin xyz=0 0 0 rpy=0 0 0, axis 0 1 0, limit lower=-0.4 upper=0.4 effort=0 velocity=1.0
- added joint HeadRAntenaFoot_J1: type revolute, parent RAntena, child HeadRAntenaFoot_J1, origin xyz=-0.0279 -0.0202 0.1006 rpy=0 0 0, axis 1 0 0, limit lower=-0.4 upper=0.4 effort=0 velocity=1.0
- added joint HeadRAntenaFoot_J2: type revolute, parent HeadRAntenaFoot_J1, child HeadRAntenaFoot_J2, origin xyz=0 0 0 rpy=0 0 0, axis 0 1 0, limit lower=-0.4 upper=0.4 effort=0 velocity=1.0
- added joint HeadRAntena_J1: type revolute, parent Head, child HeadRAntena_J1, origin xyz=-0.0168 -0.1029 0.0226 rpy=0 0 0, axis 1 0 0, limit lower=-0.4 upper=0.4 effort=0 velocity=1.0
- added joint HeadRAntena_J2: type revolute, parent HeadRAntena_J1, child HeadRAntena_J2, origin xyz=0 0 0 rpy=0 0 0, axis 0 1 0, limit lower=-0.4 upper=0.4 effort=0 velocity=1.0
- added joint LAntena: type revolute, parent HeadLAntena_J2, child LAntena, origin xyz=0 0 0 rpy=0 0 0, axis 0 0 1, limit lower=-0.2 upper=0.2 effort=0 velocity=1.0
- added joint LAntenaFoot: type revolute, parent HeadLAntenaFoot_J2, child LAntenaFoot, origin xyz=0 0 0 rpy=0 0 0, axis 0 0 1, limit lower=-0.2 upper=0.2 effort=0 velocity=1.0
- added joint LBFoot: type revolute, parent ThoraxLBFoot_J2, child LBFoot, origin xyz=0 0 0 rpy=0 0 0, axis 0 0 1, limit lower=-0.2 upper=0.2 effort=0 velocity=1.0
- added joint LBFootSphere: type fixed, parent LBFoot, child LBFootSphere, origin xyz=0.0840 0.0771 -0.1303 rpy=0 0 0
- added joint LBShank: type revolute, parent ThoraxLBShank_J2, child LBShank, origin xyz=0 0 0 rpy=0 0 0, axis 0 0 1, limit lower=-0.2 upper=0.2 effort=0 velocity=1.0
- added joint LBThigh: type revolute, parent ThoraxLBThigh_J2, child LBThigh, origin xyz=0 0 0 rpy=0 0 0, axis 0 0 1, limit lower=-0.2 upper=0.2 effort=0 velocity=1.0
- added joint LFFoot: type revolute, parent ThoraxLFFoot_J2, child LFFoot, origin xyz=0 0 0 rpy=0 0 0, axis 0 0 1, limit lower=-0.2 upper=0.2 effort=0 velocity=1.0
- added joint LFFootSphere: type fixed, parent LFFoot, child LFFootSphere, origin xyz=0.0724 -0.0430 -0.118 rpy=0 0 0
- added joint LFShank: type revolute, parent ThoraxLFShank_J2, child LFShank, origin xyz=0 0 0 rpy=0 0 0, axis 0 0 1, limit lower=-0.2 upper=0.2 effort=0 velocity=1.0
- added joint LFThigh: type revolute, parent ThoraxLFThigh_J2, child LFThigh, origin xyz=0 0 0 rpy=0 0 0, axis 0 0 1, limit lower=-0.2 upper=0.2 effort=0 velocity=1.0
- added joint LMFoot: type revolute, parent ThoraxLMFoot_J2, child LMFoot, origin xyz=0 0 0 rpy=0 0 0, axis 0 0 1, limit lower=-0.2 upper=0.2 effort=0 velocity=1.0
- added joint LMFootSphere: type fixed, parent LMFoot, child LMFootSphere, origin xyz=0.0925 0.0314 -0.1266 rpy=0 0 0
- added joint LMShank: type revolute, parent ThoraxLMShank_J2, child LMShank, origin xyz=0 0 0 rpy=0 0 0, axis 0 0 1, limit lower=-0.2 upper=0.2 effort=0 velocity=1.0
- added joint LMThigh: type revolute, parent ThoraxLMThigh_J2, child LMThigh, origin xyz=0 0 0 rpy=0 0 0, axis 0 0 1, limit lower=-0.2 upper=0.2 effort=0 velocity=1.0
- added joint RAntena: type revolute, parent HeadRAntena_J2, child RAntena, origin xyz=0 0 0 rpy=0 0 0, axis 0 0 1, limit lower=-0.2 upper=0.2 effort=0 velocity=1.0
- added joint RAntenaFoot: type revolute, parent HeadRAntenaFoot_J2, child RAntenaFoot, origin xyz=0 0 0 rpy=0 0 0, axis 0 0 1, limit lower=-0.2 upper=0.2 effort=0 velocity=1.0
- added joint RBFoot: type revolute, parent ThoraxRBFoot_J2, child RBFoot, origin xyz=0 0 0 rpy=0 0 0, axis 0 0 1, limit lower=-0.2 upper=0.2 effort=0 velocity=1.0
- added joint RBFootSphere: type fixed, parent RBFoot, child RBFootSphere, origin xyz=-0.0852 0.0768 -0.1296 rpy=0 0 0
- added joint RBShank: type revolute, parent ThoraxRBShank_J2, child RBShank, origin xyz=0 0 0 rpy=0 0 0, axis 0 0 1, limit lower=-0.2 upper=0.2 effort=0 velocity=1.0
- added joint RBThigh: type revolute, parent ThoraxRBThigh_J2, child RBThigh, origin xyz=0 0 0 rpy=0 0 0, axis 0 0 1, limit lower=-0.2 upper=0.2 effort=0 velocity=1.0
- added joint RFFoot: type revolute, parent ThoraxRFFoot_J2, child RFFoot, origin xyz=0 0 0 rpy=0 0 0, axis 0 0 1, limit lower=-0.2 upper=0.2 effort=0 velocity=1.0
- added joint RFFootSphere: type fixed, parent RFFoot, child RFFootSphere, origin xyz=-0.0729 -0.0412 -0.1177 rpy=0 0 0
- added joint RFShank: type revolute, parent ThoraxRFShank_J2, child RFShank, origin xyz=0 0 0 rpy=0 0 0, axis 0 0 1, limit lower=-0.2 upper=0.2 effort=0 velocity=1.0
- added joint RFThigh: type revolute, parent ThoraxRFThigh_J2, child RFThigh, origin xyz=0 0 0 rpy=0 0 0, axis 0 0 1, limit lower=-0.2 upper=0.2 effort=0 velocity=1.0
- added joint RMFoot: type revolute, parent ThoraxRMFoot_J2, child RMFoot, origin xyz=0 0 0 rpy=0 0 0, axis 0 0 1, limit lower=-0.2 upper=0.2 effort=0 velocity=1.0
- added joint RMFootSphere: type fixed, parent RMFoot, child RMFootSphere, origin xyz=-0.0923 0.0307 -0.1263 rpy=0 0 0
- added joint RMShank: type revolute, parent ThoraxRMShank_J2, child RMShank, origin xyz=0 0 0 rpy=0 0 0, axis 0 0 1, limit lower=-0.2 upper=0.2 effort=0 velocity=1.0
- added joint RMThigh: type revolute, parent ThoraxRMThigh_J2, child RMThigh, origin xyz=0 0 0 rpy=0 0 0, axis 0 0 1, limit lower=-0.2 upper=0.2 effort=0 velocity=1.0
- added joint ThoraxAbdomen_J1: type revolute, parent Thorax, child ThoraxAbdomen_J1, origin xyz=0 0.15853 0.19806 rpy=0 0 0, axis 1 0 0, limit lower=-0.2 upper=0.2 effort=0 velocity=1.0
- added joint ThoraxAbdomen_J2: type revolute, parent ThoraxAbdomen_J1, child ThoraxAbdomen_J2, origin xyz=0 0 0 rpy=0 0 0, axis 0 1 0, limit lower=-0.2 upper=0.2 effort=0 velocity=1.0
- added joint ThoraxHead_J1: type revolute, parent Thorax, child ThoraxHead_J1, origin xyz=0 -0.06471 0.21279 rpy=0 0 0, axis 1 0 0, limit lower=-0.2 upper=0.2 effort=0 velocity=1.0
- added joint ThoraxHead_J2: type revolute, parent ThoraxHead_J1, child ThoraxHead_J2, origin xyz=0 0 0 rpy=0 0 0, axis 0 1 0, limit lower=-0.2 upper=0.2 effort=0 velocity=1.0
- added joint ThoraxLBFoot_J1: type revolute, parent LBShank, child ThoraxLBFoot_J1, origin xyz=0.0387 0.0341 -0.0900 rpy=0 0 0, axis 1 0 0, limit lower=-0.4 upper=0.4 effort=0 velocity=1.0
- added joint ThoraxLBFoot_J2: type revolute, parent ThoraxLBFoot_J1, child ThoraxLBFoot_J2, origin xyz=0 0 0 rpy=0 0 0, axis 0 1 0, limit lower=-0.4 upper=0.4 effort=0 velocity=1.0
- added joint ThoraxLBShank_J1: type revolute, parent LBThigh, child ThoraxLBShank_J1, origin xyz=0.1238 0.1183 0.0330 rpy=0 0 0, axis 1 0 0, limit lower=-0.4 upper=0.4 effort=0 velocity=1.0
- added joint ThoraxLBShank_J2: type revolute, parent ThoraxLBShank_J1, child ThoraxLBShank_J2, origin xyz=0 0 0 rpy=0 0 0, axis 0 1 0, limit lower=-0.4 upper=0.4 effort=0 velocity=1.0
- added joint ThoraxLBThigh_J1: type revolute, parent Thorax, child ThoraxLBThigh_J1, origin xyz=0.06238 0.08879 0.18588 rpy=0 0 0, axis 1 0 0, limit lower=-0.4 upper=0.4 effort=0 velocity=1.0
- added joint ThoraxLBThigh_J2: type revolute, parent ThoraxLBThigh_J1, child ThoraxLBThigh_J2, origin xyz=0 0 0 rpy=0 0 0, axis 0 1 0, limit lower=-0.4 upper=0.4 effort=0 velocity=1.0
- added joint ThoraxLFFoot_J1: type revolute, parent LFShank, child ThoraxLFFoot_J1, origin xyz=0.0349 -0.0208 -0.0839 rpy=0 0 0, axis 1 0 0, limit lower=-0.4 upper=0.4 effort=0 velocity=1.0
- added joint ThoraxLFFoot_J2: type revolute, parent ThoraxLFFoot_J1, child ThoraxLFFoot_J2, origin xyz=0 0 0 rpy=0 0 0, axis 0 1 0, limit lower=-0.4 upper=0.4 effort=0 velocity=1.0
- added joint ThoraxLFShank_J1: type revolute, parent LFThigh, child ThoraxLFShank_J1, origin xyz=0.1217 -0.0662 0.0268 rpy=0 0 0, axis 1 0 0, limit lower=-0.4 upper=0.4 effort=0 velocity=1.0
- added joint ThoraxLFShank_J2: type revolute, parent ThoraxLFShank_J1, child ThoraxLFShank_J2, origin xyz=0 0 0 rpy=0 0 0, axis 0 1 0, limit lower=-0.4 upper=0.4 effort=0 velocity=1.0
- added joint ThoraxLFThigh_J1: type revolute, parent Thorax, child ThoraxLFThigh_J1, origin xyz=0.0743 -0.0223 0.1894 rpy=0 0 0, axis 1 0 0, limit lower=-0.4 upper=0.4 effort=0 velocity=1.0
- added joint ThoraxLFThigh_J2: type revolute, parent ThoraxLFThigh_J1, child ThoraxLFThigh_J2, origin xyz=0 0 0 rpy=0 0 0, axis 0 1 0, limit lower=-0.4 upper=0.4 effort=0 velocity=1.0
- added joint ThoraxLMFoot_J1: type revolute, parent LMShank, child ThoraxLMFoot_J1, origin xyz=0.0420 0.0142 -0.0892 rpy=0 0 0, axis 1 0 0, limit lower=-0.4 upper=0.4 effort=0 velocity=1.0
- added joint ThoraxLMFoot_J2: type revolute, parent ThoraxLMFoot_J1, child ThoraxLMFoot_J2, origin xyz=0 0 0 rpy=0 0 0, axis 0 1 0, limit lower=-0.4 upper=0.4 effort=0 velocity=1.0
- added joint ThoraxLMShank_J1: type revolute, parent LMThigh, child ThoraxLMShank_J1, origin xyz=0.1391 0.0483 0.0267 rpy=0 0 0, axis 1 0 0, limit lower=-0.4 upper=0.4 effort=0 velocity=1.0
- added joint ThoraxLMShank_J2: type revolute, parent ThoraxLMShank_J1, child ThoraxLMShank_J2, origin xyz=0 0 0 rpy=0 0 0, axis 0 1 0, limit lower=-0.4 upper=0.4 effort=0 velocity=1.0
- added joint ThoraxLMThigh_J1: type revolute, parent Thorax, child ThoraxLMThigh_J1, origin xyz=0.07469 0.03933 0.19123 rpy=0 0 0, axis 1 0 0, limit lower=-0.4 upper=0.4 effort=0 velocity=1.0
- added joint ThoraxLMThigh_J2: type revolute, parent ThoraxLMThigh_J1, child ThoraxLMThigh_J2, origin xyz=0 0 0 rpy=0 0 0, axis 0 1 0, limit lower=-0.4 upper=0.4 effort=0 velocity=1.0
- added joint ThoraxRBFoot_J1: type revolute, parent RBShank, child ThoraxRBFoot_J1, origin xyz=-0.0385 0.0344 -0.0907 rpy=0 0 0, axis 1 0 0, limit lower=-0.4 upper=0.4 effort=0 velocity=1.0
- added joint ThoraxRBFoot_J2: type revolute, parent ThoraxRBFoot_J1, child ThoraxRBFoot_J2, origin xyz=0 0 0 rpy=0 0 0, axis 0 1 0, limit lower=-0.4 upper=0.4 effort=0 velocity=1.0
- added joint ThoraxRBShank_J1: type revolute, parent RBThigh, child ThoraxRBShank_J1, origin xyz=-0.1239 0.1180 0.0334 rpy=0 0 0, axis 1 0 0, limit lower=-0.4 upper=0.4 effort=0 velocity=1.0
- added joint ThoraxRBShank_J2: type revolute, parent ThoraxRBShank_J1, child ThoraxRBShank_J2, origin xyz=0 0 0 rpy=0 0 0, axis 0 1 0, limit lower=-0.4 upper=0.4 effort=0 velocity=1.0
- added joint ThoraxRBThigh_J1: type revolute, parent Thorax, child ThoraxRBThigh_J1, origin xyz=-0.06230 0.08906 0.18543 rpy=0 0 0, axis 1 0 0, limit lower=-0.4 upper=0.4 effort=0 velocity=1.0
- added joint ThoraxRBThigh_J2: type revolute, parent ThoraxRBThigh_J1, child ThoraxRBThigh_J2, origin xyz=0 0 0 rpy=0 0 0, axis 0 1 0, limit lower=-0.4 upper=0.4 effort=0 velocity=1.0
- added joint ThoraxRFFoot_J1: type revolute, parent RFShank, child ThoraxRFFoot_J1, origin xyz=-0.0347 -0.0205 -0.0847 rpy=0 0 0, axis 1 0 0, limit lower=-0.4 upper=0.4 effort=0 velocity=1.0
- added joint ThoraxRFFoot_J2: type revolute, parent ThoraxRFFoot_J1, child ThoraxRFFoot_J2, origin xyz=0 0 0 rpy=0 0 0, axis 0 1 0, limit lower=-0.4 upper=0.4 effort=0 velocity=1.0
- added joint ThoraxRFShank_J1: type revolute, parent RFThigh, child ThoraxRFShank_J1, origin xyz=-0.1258 -0.0680 0.0258 rpy=0 0 0, axis 1 0 0, limit lower=-0.4 upper=0.4 effort=0 velocity=1.0
- added joint ThoraxRFShank_J2: type revolute, parent ThoraxRFShank_J1, child ThoraxRFShank_J2, origin xyz=0 0 0 rpy=0 0 0, axis 0 1 0, limit lower=-0.4 upper=0.4 effort=0 velocity=1.0
- added joint ThoraxRFThigh_J1: type revolute, parent Thorax, child ThoraxRFThigh_J1, origin xyz=-0.07030 -0.02046 0.18987 rpy=0 0 0, axis 1 0 0, limit lower=-0.4 upper=0.4 effort=0 velocity=1.0
- added joint ThoraxRFThigh_J2: type revolute, parent ThoraxRFThigh_J1, child ThoraxRFThigh_J2, origin xyz=0 0 0 rpy=0 0 0, axis 0 1 0, limit lower=-0.4 upper=0.4 effort=0 velocity=1.0
- added joint ThoraxRMFoot_J1: type revolute, parent RMShank, child ThoraxRMFoot_J1, origin xyz=-0.0427 0.0128 -0.0895 rpy=0 0 0, axis 1 0 0, limit lower=-0.4 upper=0.4 effort=0 velocity=1.0
- added joint ThoraxRMFoot_J2: type revolute, parent ThoraxRMFoot_J1, child ThoraxRMFoot_J2, origin xyz=0 0 0 rpy=0 0 0, axis 0 1 0, limit lower=-0.4 upper=0.4 effort=0 velocity=1.0
- added joint ThoraxRMShank_J1: type revolute, parent RMThigh, child ThoraxRMShank_J1, origin xyz=-0.1387 0.0501 0.0266 rpy=0 0 0, axis 1 0 0, limit lower=-0.4 upper=0.4 effort=0 velocity=1.0
- added joint ThoraxRMShank_J2: type revolute, parent ThoraxRMShank_J1, child ThoraxRMShank_J2, origin xyz=0 0 0 rpy=0 0 0, axis 0 1 0, limit lower=-0.4 upper=0.4 effort=0 velocity=1.0
- added joint ThoraxRMThigh_J1: type revolute, parent Thorax, child ThoraxRMThigh_J1, origin xyz=-0.07457 0.03980 0.19130 rpy=0 0 0, axis 1 0 0, limit lower=-0.4 upper=0.4 effort=0 velocity=1.0
- added joint ThoraxRMThigh_J2: type revolute, parent ThoraxRMThigh_J1, child ThoraxRMThigh_J2, origin xyz=0 0 0 rpy=0 0 0, axis 0 1 0, limit lower=-0.4 upper=0.4 effort=0 velocity=1.0
- added joint base_link_J: type fixed, parent base_link, child Thorax, origin xyz=0 0 0 rpy=0 0 0

File: urdf/friction_cone.urdf (robot description, URDF)
Before this commit: robot object, 1 links, 0 joints
Links:
- link base_link: geometry visual mesh filename=package://animals_description/meshes/cone.dae

File: urdf/plane_3d.urdf (robot description, URDF)
Before this commit: robot environment, 2 links, 1 joints
Links:
- link l_one: geometry collision mesh filename=package://animals_description/meshes/plane_3d.stl; visual mesh filename=package://animals_description/meshes/plane_3d.stl
